Commit message: 75-6f

File: ocs2_robotic_assets/resources/mobile_manipulator/realman/urdf/rm_75.urdf (robot description, URDF)
Before this commit: robot rm_75_description, 10 links, 9 joints
Links:
- link Link1: geometry collision mesh filename=package://rm_description/meshes/rm_75_6f_arm/Link1.STL; visual mesh filename=package://rm_description/meshes/rm_75_6f_arm/Link1.STL
- link Link2: geometry collision mesh filename=package://rm_description/meshes/rm_75_6f_arm/Link2.STL; visual mesh filename=package://rm_description/meshes/rm_75_6f_arm/Link2.STL
- link Link3: geometry collision mesh filename=package://rm_description/meshes/rm_75_6f_arm/Link3.STL; visual mesh filename=package://rm_description/meshes/rm_75_6f_arm/Link3.STL
- link Link4: geometry collision mesh filename=package://rm_description/meshes/rm_75_6f_arm/Link4.STL; visual mesh filename=package://rm_description/meshes/rm_75_6f_arm/Link4.STL
- link Link5: geometry collision mesh filename=package://rm_description/meshes/rm_75_6f_arm/Link5.STL; visual mesh filename=package://rm_description/meshes/rm_75_6f_arm/Link5.STL
- link Link6: geometry collision mesh filename=package://rm_description/meshes/rm_75_6f_arm/Link6.STL; visual mesh filename=package://rm_description/meshes/rm_75_6f_arm/Link6.STL
- link Link7: geometry collision mesh filename=package://rm_description/meshes/rm_75_6f_arm/Link7.STL; visual mesh filename=package://rm_description/meshes/rm_75_6f_arm/Link7.STL
- link base_link: geometry collision mesh filename=package://rm_description/meshes/rm_75_6f_arm/base_link.STL; visual mesh filename=package://rm_description/meshes/rm_75_6f_arm/base_link.STL

File: ocs2_robotic_assets/resources/mobile_manipulator/realman/urdf/rm_75_6f.urdf (robot description, URDF)
Before this commit: robot rm_75_description, 16 links, 15 joints
Links:
- link Link1: geometry collision mesh filename=package://rm_description/meshes/rm_75_6f_arm/Link1.STL; visual mesh filename=package://rm_description/meshes/rm_75_6f_arm/Link1.STL
- link Link2: geometry collision mesh filename=package://rm_description/meshes/rm_75_6f_arm/Link2.STL; visual mesh filename=package://rm_description/meshes/rm_75_6f_arm/Link2.STL
- link Link3: geometry collision mesh filename=package://rm_description/meshes/rm_75_6f_arm/Link3.STL; visual mesh filename=package://rm_description/meshes/rm_75_6f_arm/Link3.STL
- link Link4: geometry collision mesh filename=package://rm_description/meshes/rm_75_6f_arm/Link4.STL; visual mesh filename=package://rm_description/meshes/rm_75_6f_arm/Link4.STL
- link Link5: geometry collision mesh filename=package://rm_description/meshes/rm_75_6f_arm/Link5.STL; visual mesh filename=package://rm_description/meshes/rm_75_6f_arm/Link5.STL
- link Link6: geometry collision mesh filename=package://rm_description/meshes/rm_75_6f_arm/Link6.STL; visual mesh filename=package://rm_description/meshes/rm_75_6f_arm/Link6.STL
- link Link7: geometry collision mesh filename=package://rm_description/meshes/rm_75_6f_arm/Link7.STL; visual mesh filename=package://rm_description/meshes/rm_75_6f_arm/Link7.STL
- link base_link: geometry collision mesh filename=package://rm_description/meshes/rm_75_6f_arm/base_link.STL; visual mesh filename=package://rm_description/meshes/rm_75_6f_arm/base_link.STL
- link camera_connect: geometry collision mesh filename=package://rm_description/meshes/gripper/camera_connect.STL; visual mesh filename=package://rm_description/meshes/gripper/camera_connect.STL
- link gripper_Link1: geometry collision mesh filename=package://rm_description/meshes/gripper/gripper_Link1.STL; visual mesh filename=package://rm_description/meshes/gripper/gripper_Link1.STL
- link gripper_Link2: geometry collision mesh filename=package://rm_description/meshes/gripper/gripper_Link2.STL; visual mesh filename=package://rm_description/meshes/gripper/gripper_Link2.STL
- link gripper_Link3: geometry collision mesh filename=package://rm_description/meshes/gripper/gripper_Link3.STL; visual mesh filename=package://rm_description/meshes/gripper/gripper_Link3.STL
- link gripper_Link4: geometry collision mesh filename=package://rm_description/meshes/gripper/gripper_Link4.STL; visual mesh filename=package://rm_description/meshes/gripper/gripper_Link4.STL
- link gripper_base_link: geometry collision mesh filename=package://rm_description/meshes/gripper/gripper_base_link.S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; visual mesh filename=package://rm_description/meshes/gripper/gripper_base_link.S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

Commit message: add sphere approximation

File: ocs2_robotic_assets/resources/mobile_manipulator/realman/urdf/rm_75.urdf (robot description, URDF)
Before this commit: robot rm_75_description, 10 links, 9 joints
Links:
- link Link1: geometry collision cylinder length=0.10 radius=0.06; visual mesh filename=package://rm_description/meshes/rm_75_6f_arm/Link1.STL
- link Link2: geometry collision cylinder length=0.10 radius=0.06; visual mesh filename=package://rm_description/meshes/rm_75_6f_arm/Link2.STL
- link Link3: geometry collision cylinder length=0.10 radius=0.06; visual mesh filename=package://rm_description/meshes/rm_75_6f_arm/Link3.STL
- link Link4: geometry collision cylinder length=0.10 radius=0.06; visual mesh filename=package://rm_description/meshes/rm_75_6f_arm/Link4.STL
- link Link5: geometry collision cylinder length=0.10 radius=0.06; visual mesh filename=package://rm_description/meshes/rm_75_6f_arm/Link5.STL
- link Link6: geometry collision cylinder length=0.10 radius=0.06; visual mesh filename=package://rm_description/meshes/rm_75_6f_arm/Link6.STL
- link Link7: geometry collision cylinder length=0.10 radius=0.06; visual mesh filename=package://rm_description/meshes/rm_75_6f_arm/Link7.STL
- link base_link: geometry collision cylinder length=0.0012 radius=0.0006; visual mesh filename=package://rm_description/meshes/rm_75_6f_arm/base_link.STL

File: ocs2_robotic_assets/resources/mobile_manipulator/realman/urdf/rm_75_6f_description.urdf (robot description, URDF)
Before this commit: robot rm_75_description, 16 links, 15 joints
Links:
- removed link realman_tip
- removed link world
- added link gripper_tip_link
- added link hand_link
- link Link1: geometry collision cylinder length=0.1015 radius=0.08; visual mesh filename=file://$(find rm_description)/meshes/rm_75_6f_arm/Link1.STL
- link Link2: geometry collision cylinder length=0.1525 radius=0.06; visual mesh filename=file://$(find rm_description)/meshes/rm_75_6f_arm/Link2.STL
- link Link3: geometry collision cylinder length=0.125 radius=0.08; visual mesh filename=file://$(find rm_description)/meshes/rm_75_6f_arm/Link3.STL
- link Link4: geometry collision cylinder length=0.1285 radius=0.06; visual mesh filename=file://$(find rm_description)/meshes/rm_75_6f_arm/Link4.STL
- link Link5: geometry collision cylinder length=0.0815 radius=0.08; visual mesh filename=file://$(find rm_description)/meshes/rm_75_6f_arm/Link5.STL
- link Link6: geometry collision cylinder length=0.160 radius=0.06; visual mesh filename=file://$(find rm_description)/meshes/rm_75_6f_arm/Link6.STL
- link Link7: geometry collision cylinder length=0.125 radius=0.02; visual mesh filename=file://$(find rm_description)/meshes/rm_75_6f_arm/Link7.STL
- link base_link: geometry collision cylinder length=0.0012 radius=0.0006; visual mesh filename=file://$(find rm_description)/meshes/rm_75_6f_arm/base_link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
- link camera_connect: geometry collision mesh filename=file://$(find rm_description)/meshes/gripper/camera_connect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; visual mesh filename=file://$(find rm_description)/meshes/gripper/camera_connect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
- link gripper_Link1: geometry collision mesh filename=file://$(find rm_description)/meshes/gripper/gripper_Link1.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; visual mesh filename=file://$(find rm_description)/meshes/gripper/gripper_Link1.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
- link gripper_Link2: geometry collision mesh filename=file://$(find rm_description)/meshes/gripper/gripper_Link2.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; visual mesh filename=file://$(find rm_description)/meshes/gripper/gripper_Link2.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
- link gripper_Link3: geometry collision mesh filename=file://$(find rm_description)/meshes/gripper/gripper_Link3.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; visual mesh filename=file://$(find rm_description)/meshes/gripper/gripper_Link3.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
- link gripper_Link4: geometry collision mesh filename=file://$(find rm_description)/meshes/gripper/gripper_Link4.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; visual mesh filename=file://$(find rm_description)/meshes/gripper/gripper_Link4.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
- link gripper_base_link: geometry collision mesh filename=file://$(find rm_description)/meshes/gripper/gripper_base_l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; visual mesh filename=file://$(find rm_description)/meshes/gripper/gripper_base_l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
Joints:
- removed joint tip_joint
- removed joint world_joint
- added joint gripper_tip_joint: type fixed, parent Link7, child gripper_tip_link, origin xyz=0 0 0.1522 rpy=0 0 0
- added joint hand_camera_joint: type fixed, parent gripper_tip_link, child hand_link, origin xyz=9.118397057093950708e-02 -1.184690085767839060e-02 -1.088632721090737610e-01 rpy=-3.141592653589793 -1.5707963267948966 0.0
- joint gripper_joint1: axis (none) -> 1 0 0; limit (none) -> lower=-1.5708 upper=1.5708 effort=100 velocity=1; type fixed -> revolute
- joint gripper_joint2: axis (none) -> -1 0 0; limit (none) -> lower=-1.5708 upper=1.5708 effort=100 velocity=1; mimic (none) -> joint=gripper_joint1 multiplier=1 offset=0; type fixed -> revolute
- joint gripper_joint3: axis (none) -> 1 0 0; limit (none) -> lower=-1.5708 upper=1.5708 effort=100 velocity=1; type fixed -> revolute
- joint gripper_joint4: axis (none) -> -1 0 0; limit (none) -> lower=-1.5708 upper=1.5708 effort=100 velocity=1; mimic (none) -> joint=gripper_joint3 multiplier=1 offset=0; type fixed -> revolute

File: ocs2_robotic_assets/resources/mobile_manipulator/realman/urdf/rm_75_6f_description_1.urdf (robot description, URDF)
Before this commit: robot rm_75_description, 16 links, 15 joints
Links:
- removed link realman_tip
- removed link world
- added link gripper_tip_link
- added link hand_link
- link Link1: mass 0.593563458735581 -> 0.59356; geometry collision mesh filename=file://$(find rm_description)/meshes/rm_75_6f_arm/Link1.STL; visual mesh filename=file://$(find rm_description)/meshes/rm_75_6f_arm/Link1.STL
- link Link2: mass 0.432849770310974 -> 0.43285; geometry collision mesh filename=file://$(find rm_description)/meshes/rm_75_6f_arm/Link2.STL; visual mesh filename=file://$(find rm_description)/meshes/rm_75_6f_arm/Link2.STL
- link Link3: mass 0.431325495678459 -> 0.43132; geometry collision mesh filename=file://$(find rm_description)/meshes/rm_75_6f_arm/Link3.STL; visual mesh filename=file://$(find rm_description)/meshes/rm_75_6f_arm/Link3.STL
- link Link4: mass 0.289633681619295 -> 0.28963; geometry collision mesh filename=file://$(find rm_description)/meshes/rm_75_6f_arm/Link4.STL; visual mesh filename=file://$(find rm_description)/meshes/rm_75_6f_arm/Link4.STL
- link Link5: mass 0.239419768320061 -> 0.23941; geometry collision mesh filename=file://$(find rm_description)/meshes/rm_75_6f_arm/Link5.STL; visual mesh filename=file://$(find rm_description)/meshes/rm_75_6f_arm/Link5.STL
- link Link6: mass 0.218799761431682 -> 0.21879; geometry collision mesh filename=file://$(find rm_description)/meshes/rm_75_6f_arm/Link6.STL; visual mesh filename=file://$(find rm_description)/meshes/rm_75_6f_arm/Link6.STL
- link Link7: mass 0.0649018034311231 -> 0.14433; geometry collision mesh filename=file://$(find rm_description)/meshes/rm_75_6f_arm/Link7.STL; visual mesh filename=file://$(find rm_description)/meshes/rm_75_6f_arm/Link7.STL
- link base_link: mass 0.841071174772543 -> 0.84105; geometry collision mesh filename=file://$(find rm_description)/meshes/rm_75_6f_arm/base_link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; visual mesh filename=file://$(find rm_description)/meshes/rm_75_6f_arm/base_link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
- link camera_connect: geometry collision mesh filename=file://$(find rm_description)/meshes/gripper/camera_connect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; visual mesh filename=file://$(find rm_description)/meshes/gripper/camera_connect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
- link gripper_Link1: geometry collision mesh filename=file://$(find rm_description)/meshes/gripper/gripper_Link1.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; visual mesh filename=file://$(find rm_description)/meshes/gripper/gripper_Link1.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
- link gripper_Link2: geometry collision mesh filename=file://$(find rm_description)/meshes/gripper/gripper_Link2.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; visual mesh filename=file://$(find rm_description)/meshes/gripper/gripper_Link2.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
- link gripper_Link3: geometry collision mesh filename=file://$(find rm_description)/meshes/gripper/gripper_Link3.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; visual mesh filename=file://$(find rm_description)/meshes/gripper/gripper_Link3.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
- link gripper_Link4: geometry collision mesh filename=file://$(find rm_description)/meshes/gripper/gripper_Link4.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; visual mesh filename=file://$(find rm_description)/meshes/gripper/gripper_Link4.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
- link gripper_base_link: geometry collision mesh filename=file://$(find rm_description)/meshes/gripper/gripper_base_l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; visual mesh filename=file://$(find rm_description)/meshes/gripper/gripper_base_l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
Joints:
- removed joint tip_joint
- removed joint world_joint
- added joint gripper_tip_joint: type fixed, parent Link7, child gripper_tip_link, origin xyz=0 0 0.1522 rpy=0 0 0
- added joint hand_camera_joint: type fixed, parent gripper_tip_link, child hand_link, origin xyz=9.118397057093950708e-02 -1.184690085767839060e-02 -1.088632721090737610e-01 rpy=-3.141592653589793 -1.5707963267948966 0.0
- joint gripper_joint1: axis (none) -> 1 0 0; limit (none) -> lower=-1.5708 upper=1.5708 effort=100 velocity=1; type fixed -> revolute
- joint gripper_joint2: axis (none) -> -1 0 0; limit (none) -> lower=-1.5708 upper=1.5708 effort=100 velocity=1; mimic (none) -> joint=gripper_joint1 multiplier=1 offset=0; type fixed -> revolute
- joint gripper_joint3: axis (none) -> 1 0 0; limit (none) -> lower=-1.5708 upper=1.5708 effort=100 velocity=1; type fixed -> revolute
- joint gripper_joint4: axis (none) -> -1 0 0; limit (none) -> lower=-1.5708 upper=1.5708 effort=100 velocity=1; mimic (none) -> joint=gripper_joint3 multiplier=1 offset=0; type fixed -> revolute
- joint joint1: limit lower=-3.1 upper=3.1 effort=60 velocity=3.14 -> lower=-3.107 upper=3.107 effort=100 velocity=1
- joint joint2: limit lower=-2.268 upper=2.268 effort=60 velocity=3.14 -> lower=-2.269 upper=2.269 effort=100 velocity=1
- joint joint3: limit lower=-3.1 upper=3.1 effort=30 velocity=3.92 -> lower=-3.107 upper=3.107 effort=100 velocity=1
- joint joint4: limit lower=-2.355 upper=2.355 effort=30 velocity=3.92 -> lower=-2.356 upper=2.356 effort=100 velocity=1
- joint joint5: limit lower=-3.1 upper=3.1 effort=10 velocity=3.92 -> lower=-3.107 upper=3.107 effort=100 velocity=1
- joint joint6: limit lower=-2.233 upper=2.233 effort=10 velocity=3.92 -> lower=-2.234 upper=2.234 effort=100 velocity=1
- joint joint7: limit lower=-6.28 upper=6.28 effort=10 velocity=3.92 -> lower=-6.283 upper=6.283 effort=100 velocity=1
