Commit message: traj generate

File: ocs2_robotic_assets/resources/mobile_manipulator/realman/urdf/rm_75_6f.urdf (robot description, URDF)
Before this commit: robot rm_75_description, 16 links, 15 joints
Joints:
- joint joint2: limit lower=-2.268 upper=2.268 effort=60 velocity=3.14 -> lower=-0.268 upper=0.268 effort=60 velocity=3.14
