Commit message: 2025/04/30 修改底盘与机械臂base之间的变化关系，与gazebo中保持一致

File: ocs2_robotic_assets/resources/mobile_manipulator/realhex/urdf/realhex.urdf (robot description, URDF)
Before this commit: robot realhex, 22 links, 21 joints
Joints:
- joint base_to_arm_joint: origin xyz=0 0 0.25 rpy=0 0 0 -> xyz=0.02171 0 0.36 rpy=0 0 0

Commit message: 2025/05/13 调整realhex jointPositionLimits参数

File: ocs2_robotic_assets/resources/mobile_manipulator/realhex/urdf/realhex.urdf (robot description, URDF)
Before this commit: robot realhex, 22 links, 21 joints
Joints:
- joint end_effector_joint: origin xyz=0 0 0.1 rpy=0 0 0 -> xyz=0 0 0 rpy=0 0 0

Commit message: task.info线程数和优先级，需要设置用户权限来enable

File: ocs2_robotic_assets/resources/mobile_manipulator/realhex/urdf/realhex.urdf (robot description, URDF)
Before this commit: robot realhex, 22 links, 21 joints
Links:
- removed link arm_base_link
- added link mobile_base, mass 0.88922; collision mesh filename=package://ocs2_robotic_assets/resources/mobile_manipulator/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; visual mesh filename=package://ocs2_robotic_assets/resources/mobile_manipulator/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
- link base_link: mass 0.88922 -> 0.84105
Joints:
- joint base_to_arm_joint: child arm_base_link -> base_link; parent base_link -> mobile_base
- joint blc_Joint: parent base_link -> mobile_base
- joint brc_Joint: parent base_link -> mobile_base
- joint flc_Joint: parent base_link -> mobile_base
- joint frc_Joint: parent base_link -> mobile_base
- joint frontback_joint: parent base_link -> mobile_base
- joint joint1: parent arm_base_link -> base_link
- joint logo_joint: parent base_link -> mobile_base
- joint lw_Joint: parent base_link -> mobile_base
- joint parts_joint: parent base_link -> mobile_base
- joint plus_joint: parent base_link -> mobile_base
- joint print_joint: parent base_link -> mobile_base
- joint rw_Joint: parent base_link -> mobile_base
- joint up_joint: parent base_link -> mobile_base

Commit message: change mobile base

File: ocs2_robotic_assets/resources/mobile_manipulator/realhex/urdf/realhex.urdf (robot description, URDF)
Before this commit: robot realhex, 22 links, 21 joints
Links:
- removed link arm_base_link
- link base_link: mass 0.88922 -> 0.84105
Joints:
- joint base_to_arm_joint: child arm_base_link -> base_link; parent base_link -> mobile_base
- joint blc_Joint: parent base_link -> mobile_base
- joint brc_Joint: parent base_link -> mobile_base
- joint end_effector_joint: origin xyz=0 0 0 rpy=0 0 0 -> xyz=0 0 0.1522 rpy=0 0 0
- joint flc_Joint: parent base_link -> mobile_base
- joint frc_Joint: parent base_link -> mobile_base
- joint frontback_joint: parent base_link -> mobile_base
- joint joint1: parent arm_base_link -> base_link
- joint logo_joint: parent base_link -> mobile_base
- joint lw_Joint: parent base_link -> mobile_base
- joint parts_joint: parent base_link -> mobile_base
- joint plus_joint: parent base_link -> mobile_base
- joint print_joint: parent base_link -> mobile_base
- joint rw_Joint: parent base_link -> mobile_base
- joint up_joint: parent base_link -> mobile_base
